File: paper/background/starter_board/test_module_starter.kicad_pcb (KiCad board)
At the start: 2 copper layers, 145.1 x 109 mm, 14 parts, among them J1 Barrel_Jack_12V, M1 ERM_Motor, M2 Stepper_4wire, M3 Servo_3pin, U1 D24V22F5_Buck, U2 Pi_Pico_W, U3 DRV2605L_Breakout, U4 DRV8871_Breakout, U5 Tic_T500

Commit message: Rebuild starter board with real vendor component packages (PR #25)
Parts:
- C1, C2, C3: footprint powder_doser_proxies:Cap_Polar -> powder_doser_parts:Cap_Polar
- J1: footprint powder_doser_proxies:Barrel_Jack_12V -> powder_doser_parts:Barrel_Jack_12V
- M1: footprint powder_doser_proxies:ERM_Motor -> powder_doser_parts:ERM_Motor
- M2: footprint powder_doser_proxies:Stepper_4wire -> powder_doser_parts:Stepper_4wire
- M3: footprint powder_doser_proxies:Servo_3pin -> powder_doser_parts:Servo_3pin
- SOL1: footprint powder_doser_proxies:Solenoid -> powder_doser_parts:Solenoid
- SR1: footprint powder_doser_proxies:Shunt_Regulator -> powder_doser_parts:Shunt_Regulator
- U1: footprint powder_doser_proxies:D24V22F5_Buck -> powder_doser_parts:D24V22F5_Buck
- U2: footprint powder_doser_proxies:Pi_Pico_W -> powder_doser_parts:Pi_Pico_W
- U3: footprint powder_doser_proxies:DRV2605L_Breakout -> powder_doser_parts:DRV2605L_Breakout
- U4: footprint powder_doser_proxies:DRV8871_Breakout -> powder_doser_parts:DRV8871_Breakout
- U5: footprint powder_doser_proxies:Tic_T500 -> powder_doser_parts:Tic_T500
- moved M2 159.9 mm to (285.0, 145.0)
- moved M3 150.3 mm to (210.0, 215.0)
- moved SOL1 146.3 mm to (275.0, 100.0)
- moved C3 143.3 mm to (210.0, 195.0)
- moved M1 139.8 mm to (275.0, 50.0)
- moved SR1 131.0 mm to (175.0, 195.0)
- moved U5 126.2 mm to (210.0, 140.0)
- moved U4 114.2 mm to (210.0, 90.0)
- moved U3 106.9 mm to (210.0, 40.0)
- moved C2 61.8 mm to (30.0, 120.0)
- moved U2 60.4 mm to (110.0, 50.0)
- moved C1 52.2 mm to (30.0, 100.0)
- moved U1 38.1 mm to (30.0, 70.0)
- moved J1 25.0 mm to (30.0, 40.0)
Other:
- board size 145.1 x 109 mm -> 278.7 x 198.6 mm
