File: paper/background/starter_board/test_module_unplaced.kicad_pcb (KiCad board)
At the start: 2 copper layers, 79.8 x 117.7 mm, 14 parts, among them J1 Barrel_Jack_12V, M1 ERM_Motor, M2 Stepper_4wire, M3 Servo_3pin, U1 D24V22F5_Buck, U2 Pi_Pico_W, U3 DRV2605L_Breakout, U4 DRV8871_Breakout, U5 Tic_T500

Commit message: Implement Edison feedback: domain/cluster/edge-aware board placement
Parts:
- moved M3 119.2 mm to (232.9, 45.5)
- moved U2 114.8 mm to (217.8, 45.5)
- moved U3 91.9 mm to (216.8, 8.76)
- moved M1 91.2 mm to (230.9, 8.76)
- moved U4 69.4 mm to (146.3, 26.8)
- moved SR1 65.5 mm to (147.4, 52.1)
- moved U5 57.1 mm to (186.5, 52.1)
- moved M2 50.4 mm to (131.0, 52.1)
- moved U1 47.8 mm to (163.0, 6.38)
- moved SOL1 47.1 mm to (131.0, 26.8)
- moved C2 36.8 mm to (176.1, 6.38)
- moved J1 36.8 mm to (136.1, 6.38)
- moved C3 23.3 mm to (166.2, 52.1)
- moved C1 21.7 mm to (149.9, 6.38)
Other:
- board size 79.8 x 117.7 mm -> 116.6 x 82 mm
Changed lines of the file:
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@@
   (net 20 "VIB_B")
   (footprint "Connector_BarrelJack:BarrelJack_Horizontal" (version 20221018) (generator kiutils) (layer "F.Cu")
-    (at 99.32 6.383333333333334 0)
+    (at 136.10999999999999 6.383333333333334 0)
     (descr "Powder-doser starter-board part; real land pattern(s): Connector_BarrelJack:BarrelJack_Horizontal")
     (fp_text reference "J1" (at 0 -6.883333333333334 0) (layer "F.SilkS")
@@
   )
   (footprint "powder_doser_parts:D24V22F5_Buck" (version 20221018) (generator kiutils) (layer "F.Cu")
-    (at 115.16999999999999 6.16 0)
+    (at 162.95999999999998 6.383333333333334 0)
     (descr "Powder-doser starter-board part; real land pattern(s): Connector_PinHeader_2.54mm:PinHeader_1x04_P2.54mm_Vertical")
     (fp_text reference "U1" (at 0 -6.66 0) (layer "F.SilkS")
@@
   )
   (footprint "Capacitor_THT:CP_Radial_D8.0mm_P3.50mm" (version 20221018) (generator kiutils) (layer "F.Cu")
-    (at 128.26999999999998 4.75 0)
+    (at 149.85999999999999 6.383333333333334 0)
     (descr "Powder-doser starter-board part; real land pattern(s): Capacitor_THT:CP_Radial_D8.0mm_P3.50mm")
     (fp_text reference "C1" (at 0 -5.25 0) (layer "F.SilkS")
@@
   )
   (footprint "Capacitor_THT:CP_Radial_D8.0mm_P3.50mm" (version 20221018) (generator kiutils) (layer "F.Cu")
-    (at 139.26999999999998 4.75 0)
+    (at 176.06 6.383333333333334 0)
     (descr "Powder-doser starter-board part; real land pattern(s): Capacitor_THT:CP_Radial_D8.0mm_P3.50mm")
     (fp_text reference "C2" (at 0 -5.25 0) (layer "F.SilkS")
@@
   )
   (footprint "powder_doser_parts:Pi_Pico_W" (version 20221018) (generator kiutils) (layer "F.Cu")
-    (at 103.05999999999999 40.74666666666667 0)
+    (at 217.77999999999997 45.49000000000001 0)
     (descr "Powder-doser starter-board part; real land pattern(s): Connector_PinHeader_2.54mm:PinHeader_1x20_P2.54mm_Vertical")
     (fp_text reference "U2" (at 0 -26.980000000000004 0) (layer "F.SilkS")
@@
   )
   (footprint "powder_doser_parts:DRV2605L_Breakout" (version 20221018) (generator kiutils) (layer "F.Cu")
-    (at 126.03999999999999 23.02166666666667 0)
+    (at 216.77999999999997 8.755 0)
     (descr "Powder-doser starter-board part; real land pattern(s): Connector_PinHeader_2.54mm:PinHeader_1x02_P2.54mm_Vertical, Connector_PinHeader_2.54mm:PinHeader_1x06_P2.54mm_Vertical")
     (fp_text reference "U3" (at 0 -9.255 0) (layer "F.SilkS")
@@
   )
   (footprint "Connector_PinHeader_2.54mm:PinHeader_1x02_P2.54mm_Vertical" (version 20221018) (generator kiutils) (layer "F.Cu")
-    (at 140.13 17.886666666666667 0)
+    (at 230.86999999999998 8.755 0)
     (descr "Powder-doser starter-board part; real land pattern(s): Connector_PinHeader_2.54mm:PinHeader_1x02_P2.54mm_Vertical")
     (fp_text reference "M1" (at 0 -4.12 0) (layer "F.SilkS")
@@
   )
   (footprint "powder_doser_parts:DRV8871_Breakout" (version 20221018) (generator kiutils) (layer "F.Cu")
-    (at 103.33 81.29166666666667 0)
+    (at 146.32 26.831666666666667 0)
     (descr "Powder-doser starter-board part; real land pattern(s): Connector_PinHeader_2.54mm:PinHeader_1x03_P2.54mm_Vertical, Connector_PinHeader_2.54mm:PinHeader_1x04_P2.54mm_Vertical")
     (fp_text reference "U4" (at 0 -13.065 0) (layer "F.SilkS")
@@
   )
   (footprint "Connector_PinHeader_2.54mm:PinHeader_1x02_P2.54mm_Vertical" (version 20221018) (generator kiutils) (layer "F.Cu")
-    (at 118.69 72.34666666666668 0)
+    (at 130.95999999999998 26.831666666666667 0)
     (descr "Powder-doser starter-board part; real land pattern(s): Connector_PinHeader_2.54mm:PinHeader_1x02_P2.54mm_Vertical")
     (fp_text reference "SOL1" (at 0 -4.12 0) (layer "F.SilkS")
@@
   )
   (footprint "powder_doser_parts:Tic_T500" (version 20221018) (generator kiutils) (layer "F.Cu")
-    (at 136.58999999999997 79.96666666666667 0)
+    (at 186.48999999999998 52.13666666666667 0)
     (descr "Powder-doser starter-board part; real land pattern(s): Connector_PinHeader_2.54mm:PinHeader_1x06_P2.54mm_Vertical, Connector_PinHeader_2.54mm:PinHeader_1x08_P2.54mm_Vertical")
     (fp_text reference "U5" (at 0 -11.74 0) (layer "F.SilkS")
@@
   )
   (footprint "Capacitor_THT:CP_Radial_D8.0mm_P3.50mm" (version 20221018) (generator kiutils) (layer "F.Cu")
-    (at 156.89 73.47666666666667 0)
+    (at 166.19 52.13666666666667 0)
     (descr "Powder-doser starter-board part; real land pattern(s): Capacitor_THT:CP_Radial_D8.0mm_P3.50mm")
     (fp_text reference "C3" (at 0 -5.25 0) (layer "F.SilkS")
@@
   )
   (footprint "powder_doser_parts:Shunt_Regulator" (version 20221018) (generator kiutils) (layer "F.Cu")
-    (at 104.38499999999999 101.51666666666667 0)
+    (at 147.375 52.13666666666667 0)
     (descr "Powder-doser starter-board part; real land pattern(s): Connector_PinHeader_2.54mm:PinHeader_1x04_P2.54mm_Vertical")
     (fp_text reference "SR1" (at 0 -6.66 0) (layer "F.SilkS")
@@
   )
   (footprint "Connector_PinHeader_2.54mm:PinHeader_1x04_P2.54mm_Vertical" (version 20221018) (generator kiutils) (layer "F.Cu")
-    (at 120.8 101.51666666666667 0)
+    (at 130.95999999999998 52.13666666666667 0)
     (descr "Powder-doser starter-board part; real land pattern(s): Connector_PinHeader_2.54mm:PinHeader_1x04_P2.54mm_Vertical")
     (fp_text reference "M2" (at 0 -6.66 0) (layer "F.SilkS")
@@
   )
   (footprint "Connector_PinHeader_2.54mm:PinHeader_1x03_P2.54mm_Vertical" (version 20221018) (generator kiutils) (layer "F.Cu")
-    (at 127.0 100.24666666666667 0)
+    (at 232.86999999999998 45.49000000000001 0)
     (descr "Powder-doser starter-board part; real land pattern(s): Connector_PinHeader_2.54mm:PinHeader_1x03_P2.54mm_Vertical")
     (fp_text reference "M3" (at 0 -5.390000000000001 0) (layer "F.SilkS")
@@
     )
   )
-  (gr_line (start -5.0 -5.0) (end 74.82 -5.0) (layer "Edge.Cuts") (width 0.1))
-  (gr_line (start 74.82 -5.0) (end 74.82 112.67666666666666) (layer "Edge.Cuts") (width 0.1))
-  (gr_line (start 74.82 112.67666666666666) (end -5.0 112.67666666666666) (layer "Edge.Cuts") (width 0.1))
-  (gr_line (start -5.0 112.67666666666666) (end -5.0 -5.0) (layer "Edge.Cuts") (width 0.1))
+  (gr_line (start -5.0 -5.0) (end 111.60999999999999 -5.0) (layer "Edge.Cuts") (width 0.1))
+  (gr_line (start 111.60999999999999 -5.0) (end 111.60999999999999 76.97000000000001) (layer "Edge.Cuts") (width 0.1))
+  (gr_line (start 111.60999999999999 76.97000000000001) (end -5.0 76.97000000000001) (layer "Edge.Cuts") (width 0.1))
+  (gr_line (start -5.0 76.97000000000001) (end -5.0 -5.0) (layer "Edge.Cuts") (width 0.1))
 )

Commit message: Add Waveshare Pico-2CH-RS232 module footprint for scale integration
Parts:
- added J2: RS232_2CH_Module, powder_doser_parts:RS232_2CH_Module, F.Cu at (265.7, 45.5)
- moved M3 48.0 mm to (280.8, 45.5)
- moved U2 24.0 mm to (241.8, 45.5)
- moved C1 24.0 mm to (173.8, 6.38)
- moved C2 24.0 mm to (200.0, 6.38)
- moved C3 24.0 mm to (190.2, 52.1)
- moved J1 24.0 mm to (160.1, 6.38)
- moved M1 24.0 mm to (254.8, 8.76)
- moved M2 24.0 mm to (154.9, 52.1)
- moved SOL1 24.0 mm to (154.9, 26.8)
- moved SR1 24.0 mm to (171.4, 52.1)
- moved U1 24.0 mm to (186.9, 6.38)
- moved U3 24.0 mm to (240.8, 8.76)
- moved U4 24.0 mm to (170.3, 26.8)
- moved U5 24.0 mm to (210.5, 52.1)
Connections:
- U2 pad 11: (no net) -> RS232_1_TXD
- U2 pad 12: (no net) -> RS232_1_RXD
- U2 pad 16: (no net) -> RS232_0_TXD
- U2 pad 17: (no net) -> RS232_0_RXD
Other:
- board size 116.6 x 82 mm -> 140.6 x 82 mm
