File: paper/background/starter_board/test_module_unplaced.kicad_pcb (KiCad board)
At the start: 2 copper layers, 140.6 x 82 mm, 15 parts, among them J1 Barrel_Jack_12V, J2 RS232_2CH_Module, M1 ERM_Motor, M2 Stepper_4wire, M3 Servo_3pin, U1 D24V22F5_Buck, U2 Pi_Pico_W, U3 DRV2605L_Breakout, U4 DRV8871_Breakout, U5 Tic_T500

Commit message: Right-size unplaced board to 100x100mm; document Quilter stackup recommendation + datasheet-verification prep
Parts:
- moved C2 40.6 mm to (159.4, 6.38)
- moved C3 40.6 mm to (149.6, 52.1)
- moved J2 40.6 mm to (225.1, 45.5)
- moved M3 40.6 mm to (240.2, 45.5)
- moved SR1 40.6 mm to (130.8, 52.1)
- moved C1 40.6 mm to (133.2, 6.38)
- moved J1 40.6 mm to (119.5, 6.38)
- moved M1 40.6 mm to (214.3, 8.76)
- moved M2 40.6 mm to (114.3, 52.1)
- moved SOL1 40.6 mm to (114.3, 26.8)
- moved U1 40.6 mm to (146.3, 6.38)
- moved U2 40.6 mm to (201.2, 45.5)
- moved U3 40.6 mm to (200.2, 8.76)
- moved U4 40.6 mm to (129.7, 26.8)
- moved U5 40.6 mm to (169.9, 52.1)
Other:
- board size 140.6 x 82 mm -> 100 x 100 mm
Changed lines of the file:
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@@
   (net 24 "VIB_B")
   (footprint "Connector_BarrelJack:BarrelJack_Horizontal" (version 20221018) (generator kiutils) (layer "F.Cu")
-    (at 160.09 6.383333333333334 0)
+    (at 119.5 6.383333333333334 0)
     (descr "Powder-doser starter-board part; real land pattern(s): Connector_BarrelJack:BarrelJack_Horizontal")
     (attr through_hole)
@@
   )
   (footprint "powder_doser_parts:D24V22F5_Buck" (version 20221018) (generator kiutils) (layer "F.Cu")
-    (at 186.94 6.383333333333334 0)
+    (at 146.35 6.383333333333334 0)
     (descr "Powder-doser starter-board part; real land pattern(s): Connector_PinHeader_2.54mm:PinHeader_1x04_P2.54mm_Vertical")
     (attr through_hole)
@@
   )
   (footprint "Capacitor_THT:CP_Radial_D8.0mm_P3.50mm" (version 20221018) (generator kiutils) (layer "F.Cu")
-    (at 173.84 6.383333333333334 0)
+    (at 133.25 6.383333333333334 0)
     (descr "Powder-doser starter-board part; real land pattern(s): Capacitor_THT:CP_Radial_D8.0mm_P3.50mm")
     (attr through_hole)
@@
   )
   (footprint "Capacitor_THT:CP_Radial_D8.0mm_P3.50mm" (version 20221018) (generator kiutils) (layer "F.Cu")
-    (at 200.04000000000002 6.383333333333334 0)
+    (at 159.45 6.383333333333334 0)
     (descr "Powder-doser starter-board part; real land pattern(s): Capacitor_THT:CP_Radial_D8.0mm_P3.50mm")
     (attr through_hole)
@@
   )
   (footprint "powder_doser_parts:Pi_Pico_W" (version 20221018) (generator kiutils) (layer "F.Cu")
-    (at 241.76 45.510000000000005 0)
+    (at 201.17 45.510000000000005 0)
     (descr "Powder-doser starter-board part; real land pattern(s): Connector_PinHeader_2.54mm:PinHeader_1x20_P2.54mm_Vertical")
     (attr through_hole)
@@
   )
   (footprint "powder_doser_parts:DRV2605L_Breakout" (version 20221018) (generator kiutils) (layer "F.Cu")
-    (at 240.76 8.755 0)
+    (at 200.17 8.755 0)
     (descr "Powder-doser starter-board part; real land pattern(s): Connector_PinHeader_2.54mm:PinHeader_1x02_P2.54mm_Vertical, Connector_PinHeader_2.54mm:PinHeader_1x06_P2.54mm_Vertical")
     (attr through_hole)
@@
   )
   (footprint "Connector_PinHeader_2.54mm:PinHeader_1x02_P2.54mm_Vertical" (version 20221018) (generator kiutils) (layer "F.Cu")
-    (at 254.85 8.755 0)
+    (at 214.26 8.755 0)
     (descr "Powder-doser starter-board part; real land pattern(s): Connector_PinHeader_2.54mm:PinHeader_1x02_P2.54mm_Vertical")
     (attr through_hole)
@@
   )
   (footprint "powder_doser_parts:DRV8871_Breakout" (version 20221018) (generator kiutils) (layer "F.Cu")
-    (at 170.3 26.831666666666667 0)
+    (at 129.71 26.831666666666667 0)
     (descr "Powder-doser starter-board part; real land pattern(s): Connector_PinHeader_2.54mm:PinHeader_1x03_P2.54mm_Vertical, Connector_PinHeader_2.54mm:PinHeader_1x04_P2.54mm_Vertical")
     (attr through_hole)
@@
   )
   (footprint "Connector_PinHeader_2.54mm:PinHeader_1x02_P2.54mm_Vertical" (version 20221018) (generator kiutils) (layer "F.Cu")
-    (at 154.94 26.831666666666667 0)
+    (at 114.35 26.831666666666667 0)
     (descr "Powder-doser starter-board part; real land pattern(s): Connector_PinHeader_2.54mm:PinHeader_1x02_P2.54mm_Vertical")
     (attr through_hole)
@@
   )
   (footprint "powder_doser_parts:Tic_T500" (version 20221018) (generator kiutils) (layer "F.Cu")
-    (at 210.47 52.13666666666667 0)
+    (at 169.88 52.13666666666667 0)
     (descr "Powder-doser starter-board part; real land pattern(s): Connector_PinHeader_2.54mm:PinHeader_1x06_P2.54mm_Vertical, Connector_PinHeader_2.54mm:PinHeader_1x08_P2.54mm_Vertical")
     (attr through_hole)
@@
   )
   (footprint "Capacitor_THT:CP_Radial_D8.0mm_P3.50mm" (version 20221018) (generator kiutils) (layer "F.Cu")
-    (at 190.17000000000002 52.13666666666667 0)
+    (at 149.57999999999998 52.13666666666667 0)
     (descr "Powder-doser starter-board part; real land pattern(s): Capacitor_THT:CP_Radial_D8.0mm_P3.50mm")
     (attr through_hole)
@@
   )
   (footprint "powder_doser_parts:Shunt_Regulator" (version 20221018) (generator kiutils) (layer "F.Cu")
-    (at 171.35500000000002 52.13666666666667 0)
+    (at 130.765 52.13666666666667 0)
     (descr "Powder-doser starter-board part; real land pattern(s): Connector_PinHeader_2.54mm:PinHeader_1x04_P2.54mm_Vertical")
     (attr through_hole)
@@
   )
   (footprint "Connector_PinHeader_2.54mm:PinHeader_1x04_P2.54mm_Vertical" (version 20221018) (generator kiutils) (layer "F.Cu")
-    (at 154.94 52.13666666666667 0)
+    (at 114.35 52.13666666666667 0)
     (descr "Powder-doser starter-board part; real land pattern(s): Connector_PinHeader_2.54mm:PinHeader_1x04_P2.54mm_Vertical")
     (attr through_hole)
@@
   )
   (footprint "Connector_PinHeader_2.54mm:PinHeader_1x03_P2.54mm_Vertical" (version 20221018) (generator kiutils) (layer "F.Cu")
-    (at 280.83000000000004 45.510000000000005 0)
+    (at 240.24 45.510000000000005 0)
     (descr "Powder-doser starter-board part; real land pattern(s): Connector_PinHeader_2.54mm:PinHeader_1x03_P2.54mm_Vertical")
     (attr through_hole)
@@
   )
   (footprint "powder_doser_parts:RS232_2CH_Module" (version 20221018) (generator kiutils) (layer "F.Cu")
-    (at 265.74 45.510000000000005 0)
+    (at 225.14999999999998 45.510000000000005 0)
     (descr "Powder-doser starter-board part; real land pattern(s): Connector_PinHeader_2.54mm:PinHeader_1x20_P2.54mm_Vertical")
     (attr through_hole)
@@
     )
   )
-  (gr_line (start -5.0 -5.0) (end 135.59 -5.0) (layer "Edge.Cuts") (width 0.1))
-  (gr_line (start 135.59 -5.0) (end 135.59 77.01) (layer "Edge.Cuts") (width 0.1))
-  (gr_line (start 135.59 77.01) (end -5.0 77.01) (layer "Edge.Cuts") (width 0.1))
-  (gr_line (start -5.0 77.01) (end -5.0 -5.0) (layer "Edge.Cuts") (width 0.1))
+  (gr_line (start -5.0 -5.0) (end 95.0 -5.0) (layer "Edge.Cuts") (width 0.1))
+  (gr_line (start 95.0 -5.0) (end 95.0 95.0) (layer "Edge.Cuts") (width 0.1))
+  (gr_line (start 95.0 95.0) (end -5.0 95.0) (layer "Edge.Cuts") (width 0.1))
+  (gr_line (start -5.0 95.0) (end -5.0 -5.0) (layer "Edge.Cuts") (width 0.1))
 )
