File: paper/background/starter_board/test_module_unplaced.kicad_pcb (KiCad board)
At the start: 2 copper layers, 100 x 100 mm, 15 parts, among them J1 Barrel_Jack_12V, J2 RS232_2CH_Module, M1 ERM_Motor, M2 Stepper_4wire, M3 Servo_3pin, U1 D24V22F5_Buck, U2 Pi_Pico_W, U3 DRV2605L_Breakout, U4 DRV8871_Breakout, U5 Tic_T500

Commit message: Align starter-board KiCad trios with PR #100 scale integration (U6 RS-232 on +3V3, SCALE_TX/RX)
Regenerates both upload trios from PR #100's rev B netlist: the Waveshare
Pico-2CH-RS232 becomes U6 reached via its channel-0 4-pin TTL header
(VCC on +3V3 so the TTL swing stays inside the RP2040 abs max), wired
straight across on UART0 (GP12->TXD = SCALE_TX, GP13<-RXD = SCALE_RX);
the 40-pad J2 receptacle model and the spare GP8/GP9 channel nets are
dropped. Board is now 15 footprints / 101 pads / 75 net-assigned /
22 nets. Verified: kicad-cli netlist (75 pins, 22 nets, zero
unconnected), pcbnew DRC (0 courtyard/clearance errors, both trios),
15<->15 footprint<->symbol UUID bijection, byte-for-byte reproducible,
netlist cross-checked ref-by-ref against PR #100's PLACEMENTS
(identical 22-net set), and PR #100's ngspice RS-232 interface
analysis re-run (9/9 PASS).

Co-authored-by: Luke Blaine Winters <288785662+lbwinters@users.noreply.github.com>
Co-Authored-By: Claude Fable 5 <noreply@anthropic.com>
Parts:
- removed J2: RS232_2CH_Module, powder_doser_parts:RS232_2CH_Module
- added U6: Waveshare_2CH_RS232, powder_doser_parts:Waveshare_2CH_RS232, F.Cu at (224.9, 45.5)
- moved M3 0.48 mm to (239.8, 45.5)
Connections:
- U2 pad 11: RS232_1_TXD -> (no net)
- U2 pad 12: RS232_1_RXD -> (no net)
- U2 pad 16: RS232_0_TXD -> SCALE_TX
- U2 pad 17: RS232_0_RXD -> SCALE_RX

Commit message: Fix U6 RS-232 module footprint: restore 2x20 receptacle (mid-body 4-pin header was unpluggable)
@lbwinters caught that the generated layout placed the Waveshare
Pico-2CH-RS232 module's pin holes in the middle of its 21x52 mm body,
which would make the physical module impossible to plug in. The PR #100
alignment had adopted that PR's bench-symbol abstraction ("only its
4-pin TTL header reaches the Pico") literally, but the module's own
schematic (hardware/vendor-files/waveshare-pico-2ch-rs232) shows no
such header exists: its TTL signals live only on its 2x20
Pico-form-factor header.

U6 is again the 2x20 side receptacle the module actually plugs onto
(two real PinHeader_1x20 columns at the Pico's 17.78 mm row spacing,
as the pre-PR#100 J2 was), keeping PR #100's electrical intent:
channel 0 straight across to UART0 by board copper (GP12 -> TXD0 =
SCALE_TX, GP13 <- RXD0 = SCALE_RX), VCC (VSYS position) and the
3V3-position LED rail on +3V3, all 8 GND positions grounded,
channel 1 spare.

Board becomes 15 footprints / 137 pads / 83 net-assigned / 22 nets.
Verified: kicad-cli sch export netlist (83 pins, 22 nets, zero
unconnected, both trios), pcbnew 7.0.11 DRC (0 courtyard/clearance
errors), 15<->15 footprint<->symbol UUID bijection, byte-for-byte
reproducible, KiCad 7 20221018 format kept. Both trios + previews
regenerated; note 21, background README, and the vendor-files README
updated.

Co-authored-by: Luke Blaine Winters <288785662+lbwinters@users.noreply.github.com>
Co-Authored-By: Claude Fable 5 <noreply@anthropic.com>
Parts:
- moved M3 0.48 mm to (240.2, 45.5)
- moved U6 0.24 mm to (225.1, 45.5)
Connections:
- U6 pad 1: +3V3 -> SCALE_TX
- U6 pad 2: GND -> SCALE_RX
- U6 pad 3: SCALE_TX -> GND
- U6 pad 4: SCALE_RX -> (no net)
Changed lines of the file:
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@@
   )
   (footprint "Connector_PinHeader_2.54mm:PinHeader_1x03_P2.54mm_Vertical" (version 20221018) (generator kiutils) (layer "F.Cu")
-    (at 239.76 45.510000000000005 0)
+    (at 240.24 45.510000000000005 0)
     (descr "Powder-doser starter-board part; real land pattern(s): Connector_PinHeader_2.54mm:PinHeader_1x03_P2.54mm_Vertical")
     (attr through_hole)
@@
   )
   (footprint "powder_doser_parts:Waveshare_2CH_RS232" (version 20221018) (generator kiutils) (layer "F.Cu")
-    (at 224.91 45.510000000000005 0)
-    (descr "Powder-doser starter-board part; real land pattern(s): Connector_PinHeader_2.54mm:PinHeader_1x04_P2.54mm_Vertical")
+    (at 225.14999999999998 45.510000000000005 0)
+    (descr "Powder-doser starter-board part; real land pattern(s): Connector_PinHeader_2.54mm:PinHeader_1x20_P2.54mm_Vertical")
     (attr through_hole)
     (fp_text reference "U6" (at 0 -27.0 0) (layer "F.SilkS")
@@
       (effects (font (size 1.0 1.0) (thickness 0.15)))
     )
-    (fp_line (start -10.5 -26.0) (end 10.5 -26.0) (layer "F.Fab") (width 0.1))
-    (fp_line (start 10.5 -26.0) (end 10.5 26.0) (layer "F.Fab") (width 0.1))
-    (fp_line (start 10.5 26.0) (end -10.5 26.0) (layer "F.Fab") (width 0.1))
-    (fp_line (start -10.5 26.0) (end -10.5 -26.0) (layer "F.Fab") (width 0.1))
-    (fp_line (start -10.6 -26.1) (end 10.6 -26.1) (layer "F.SilkS") (width 0.12))
-    (fp_line (start 10.6 -26.1) (end 10.6 26.1) (layer "F.SilkS") (width 0.12))
-    (fp_line (start 10.6 26.1) (end -10.6 26.1) (layer "F.SilkS") (width 0.12))
-    (fp_line (start -10.6 26.1) (end -10.6 -26.1) (layer "F.SilkS") (width 0.12))
-    (fp_line (start -11.0 -26.5) (end 11.0 -26.5) (layer "F.CrtYd") (width 0.05))
-    (fp_line (start 11.0 -26.5) (end 11.0 26.5) (layer "F.CrtYd") (width 0.05))
-    (fp_line (start 11.0 26.5) (end -11.0 26.5) (layer "F.CrtYd") (width 0.05))
-    (fp_line (start -11.0 26.5) (end -11.0 -26.5) (layer "F.CrtYd") (width 0.05))
-    (pad "1" thru_hole rect (at 0.0 -3.81 0) (size 1.7 1.7) (drill 1) (layers *.Cu *.Mask)
+    (fp_line (start -10.74 -26.0) (end 10.74 -26.0) (layer "F.Fab") (width 0.1))
+    (fp_line (start 10.74 -26.0) (end 10.74 26.0) (layer "F.Fab") (width 0.1))
+    (fp_line (start 10.74 26.0) (end -10.74 26.0) (layer "F.Fab") (width 0.1))
+    (fp_line (start -10.74 26.0) (end -10.74 -26.0) (layer "F.Fab") (width 0.1))
+    (fp_line (start -10.84 -26.1) (end 10.84 -26.1) (layer "F.SilkS") (width 0.12))
+    (fp_line (start 10.84 -26.1) (end 10.84 26.1) (layer "F.SilkS") (width 0.12))
+    (fp_line (start 10.84 26.1) (end -10.84 26.1) (layer "F.SilkS") (width 0.12))
+    (fp_line (start -10.84 26.1) (end -10.84 -26.1) (layer "F.SilkS") (width 0.12))
+    (fp_line (start -11.24 -26.5) (end 11.24 -26.5) (layer "F.CrtYd") (width 0.05))
+    (fp_line (start 11.24 -26.5) (end 11.24 26.5) (layer "F.CrtYd") (width 0.05))
+    (fp_line (start 11.24 26.5) (end -11.24 26.5) (layer "F.CrtYd") (width 0.05))
+    (fp_line (start -11.24 26.5) (end -11.24 -26.5) (layer "F.CrtYd") (width 0.05))
+    (pad "1" thru_hole rect (at -8.89 -24.13 0) (size 1.7 1.7) (drill 1) (layers *.Cu *.Mask)
+      (net 9 "SCALE_TX") (pinfunction "TXD0"))
+    (pad "2" thru_hole oval (at -8.89 -21.59 0) (size 1.7 1.7) (drill 1) (layers *.Cu *.Mask)
+      (net 8 "SCALE_RX") (pinfunction "RXD0"))
+    (pad "3" thru_hole oval (at -8.89 -19.05 0) (size 1.7 1.7) (drill 1) (layers *.Cu *.Mask)
+      (net 4 "GND") (pinfunction "GND"))
+    (pad "4" thru_hole oval (at -8.89 -16.51 0) (size 1.7 1.7) (drill 1) (layers *.Cu *.Mask)
+      (net 0 "") (pinfunction "GP2"))
+    (pad "5" thru_hole oval (at -8.89 -13.97 0) (size 1.7 1.7) (drill 1) (layers *.Cu *.Mask)
+      (net 0 "") (pinfunction "GP3"))
+    (pad "6" thru_hole oval (at -8.89 -11.43 0) (size 1.7 1.7) (drill 1) (layers *.Cu *.Mask)
+      (net 0 "") (pinfunction "TXD1"))
+    (pad "7" thru_hole oval (at -8.89 -8.89 0) (size 1.7 1.7) (drill 1) (layers *.Cu *.Mask)
+      (net 0 "") (pinfunction "RXD1"))
+    (pad "8" thru_hole oval (at -8.89 -6.35 0) (size 1.7 1.7) (drill 1) (layers *.Cu *.Mask)
+      (net 4 "GND") (pinfunction "GND"))
+    (pad "9" thru_hole oval (at -8.89 -3.81 0) (size 1.7 1.7) (drill 1) (layers *.Cu *.Mask)
+      (net 0 "") (pinfunction "GP6"))
+    (pad "10" thru_hole oval (at -8.89 -1.27 0) (size 1.7 1.7) (drill 1) (layers *.Cu *.Mask)
+      (net 0 "") (pinfunction "GP7"))
+    (pad "11" thru_hole oval (at -8.89 1.27 0) (size 1.7 1.7) (drill 1) (layers *.Cu *.Mask)
+      (net 0 "") (pinfunction "GP8"))
+    (pad "12" thru_hole oval (at -8.89 3.81 0) (size 1.7 1.7) (drill 1) (layers *.Cu *.Mask)
+      (net 0 "") (pinfunction "GP9"))
+    (pad "13" thru_hole oval (at -8.89 6.35 0) (size 1.7 1.7) (drill 1) (layers *.Cu *.Mask)
+      (net 4 "GND") (pinfunction "GND"))
+    (pad "14" thru_hole oval (at -8.89 8.89 0) (size 1.7 1.7) (drill 1) (layers *.Cu *.Mask)
+      (net 0 "") (pinfunction "GP10"))
+    (pad "15" thru_hole oval (at -8.89 11.43 0) (size 1.7 1.7) (drill 1) (layers *.Cu *.Mask)
+      (net 0 "") (pinfunction "GP11"))
+    (pad "16" thru_hole oval (at -8.89 13.97 0) (size 1.7 1.7) (drill 1) (layers *.Cu *.Mask)
+      (net 0 "") (pinfunction "GP12"))
+    (pad "17" thru_hole oval (at -8.89 16.51 0) (size 1.7 1.7) (drill 1) (layers *.Cu *.Mask)
+      (net 0 "") (pinfunction "GP13"))
+    (pad "18" thru_hole oval (at -8.89 19.05 0) (size 1.7 1.7) (drill 1) (layers *.Cu *.Mask)
+      (net 4 "GND") (pinfunction "GND"))
+    (pad "19" thru_hole oval (at -8.89 21.59 0) (size 1.7 1.7) (drill 1) (layers *.Cu *.Mask)
+      (net 0 "") (pinfunction "GP14"))
+    (pad "20" thru_hole oval (at -8.89 24.13 0) (size 1.7 1.7) (drill 1) (layers *.Cu *.Mask)
+      (net 0 "") (pinfunction "GP15"))
+    (pad "21" thru_hole rect (at 8.89 -24.13 0) (size 1.7 1.7) (drill 1) (layers *.Cu *.Mask)
+      (net 0 "") (pinfunction "VBUS"))
+    (pad "22" thru_hole oval (at 8.89 -21.59 0) (size 1.7 1.7) (drill 1) (layers *.Cu *.Mask)
       (net 2 "+3V3") (pinfunction "VCC"))
-    (pad "2" thru_hole oval (at 0.0 -1.27 0) (size 1.7 1.7) (drill 1) (layers *.Cu *.Mask)
+    (pad "23" thru_hole oval (at 8.89 -19.05 0) (size 1.7 1.7) (drill 1) (layers *.Cu *.Mask)
       (net 4 "GND") (pinfunction "GND"))
-    (pad "3" thru_hole oval (at 0.0 1.27 0) (size 1.7 1.7) (drill 1) (layers *.Cu *.Mask)
-      (net 9 "SCALE_TX") (pinfunction "TXD"))
-    (pad "4" thru_hole oval (at 0.0 3.81 0) (size 1.7 1.7) (drill 1) (layers *.Cu *.Mask)
-      (net 8 "SCALE_RX") (pinfunction "RXD"))
+    (pad "24" thru_hole oval (at 8.89 -16.51 0) (size 1.7 1.7) (drill 1) (layers *.Cu *.Mask)
+      (net 0 "") (pinfunction "3V3_EN"))
+    (pad "25" thru_hole oval (at 8.89 -13.97 0) (size 1.7 1.7) (drill 1) (layers *.Cu *.Mask)
+      (net 2 "+3V3") (pinfunction "3V3"))
+    (pad "26" thru_hole oval (at 8.89 -11.43 0) (size 1.7 1.7) (drill 1) (layers *.Cu *.Mask)
+      (net 0 "") (pinfunction "ADC_VREF"))
+    (pad "27" thru_hole oval (at 8.89 -8.89 0) (size 1.7 1.7) (drill 1) (layers *.Cu *.Mask)
+      (net 0 "") (pinfunction "GP28"))
+    (pad "28" thru_hole oval (at 8.89 -6.35 0) (size 1.7 1.7) (drill 1) (layers *.Cu *.Mask)
+      (net 4 "GND") (pinfunction "GND"))
+    (pad "29" thru_hole oval (at 8.89 -3.81 0) (size 1.7 1.7) (drill 1) (layers *.Cu *.Mask)
+      (net 0 "") (pinfunction "GP27"))
+    (pad "30" thru_hole oval (at 8.89 -1.27 0) (size 1.7 1.7) (drill 1) (layers *.Cu *.Mask)
+      (net 0 "") (pinfunction "GP26"))
+    (pad "31" thru_hole oval (at 8.89 1.27 0) (size 1.7 1.7) (drill 1) (layers *.Cu *.Mask)
+      (net 0 "") (pinfunction "RUN"))
+    (pad "32" thru_hole oval (at 8.89 3.81 0) (size 1.7 1.7) (drill 1) (layers *.Cu *.Mask)
+      (net 0 "") (pinfunction "GP22"))
+    (pad "33" thru_hole oval (at 8.89 6.35 0) (size 1.7 1.7) (drill 1) (layers *.Cu *.Mask)
+      (net 4 "GND") (pinfunction "GND"))
+    (pad "34" thru_hole oval (at 8.89 8.89 0) (size 1.7 1.7) (drill 1) (layers *.Cu *.Mask)
+      (net 0 "") (pinfunction "GP21"))
+    (pad "35" thru_hole oval (at 8.89 11.43 0) (size 1.7 1.7) (drill 1) (layers *.Cu *.Mask)
+      (net 0 "") (pinfunction "GP20"))
+    (pad "36" thru_hole oval (at 8.89 13.97 0) (size 1.7 1.7) (drill 1) (layers *.Cu *.Mask)
+      (net 0 "") (pinfunction "GP19"))
+    (pad "37" thru_hole oval (at 8.89 16.51 0) (size 1.7 1.7) (drill 1) (layers *.Cu *.Mask)
+      (net 0 "") (pinfunction "GP18"))
+    (pad "38" thru_hole oval (at 8.89 19.05 0) (size 1.7 1.7) (drill 1) (layers *.Cu *.Mask)
+      (net 4 "GND") (pinfunction "GND"))
+    (pad "39" thru_hole oval (at 8.89 21.59 0) (size 1.7 1.7) (drill 1) (layers *.Cu *.Mask)
+      (net 0 "") (pinfunction "GP17"))
+    (pad "40" thru_hole oval (at 8.89 24.13 0) (size 1.7 1.7) (drill 1) (layers *.Cu *.Mask)
+      (net 0 "") (pinfunction "GP16"))
   )
   (gr_line (start -5.0 -5.0) (end 95.0 -5.0) (layer "Edge.Cuts") (width 0.1))

Commit message: Full physical-footprint audit: vendor-exact hole maps for all 5 carriers + barrel-jack GND fix
Re-verified every component against primary vendor geometry (PR #25 Eagle
.brd files, Pololu reg19a/tvs01a/tic03b dimension diagrams + official
tic03b drill-guide DXF, CUI PJ-102AH datasheet, Waveshare module schematic,
Pico mechanical drawing) per PR #76 review request. Fixes five unpluggable
land patterns (Tic T500 38.1x26.7 mm with all 29 real holes and correct
A2/A1 order; D24V22F5 17.8x17.8 mm PG/EN/VIN/GND/VOUT row + offset GND;
shunt regulator 28.6x20.3 mm wire terminals; DRV8871 3.5 mm terminal
blocks + 1x4 logic header; DRV2605L STEMMA QT 1x5 row with real SCL/SDA
order, EN pin dropped as nonexistent) and one wiring fault (barrel-jack
GND was on the switch lug, which floats when a plug is inserted; now on
the sleeve). Boards grow to 172 pads / 95 net-assigned / 22 nets; the
unplaced auto-place outline is re-sized 100x100 -> 110x110 mm to stay in
the 35-55% utilisation band with the real bodies. kicad-cli netlist
(95 pins, zero unconnected), pcbnew DRC (no courtyard/clearance/short
errors), 15<->15 footprint<->symbol UUID bijection, and byte-for-byte
reproducibility all re-verified on both trios.

Co-authored-by: Luke Blaine Winters <288785662+lbwinters@users.noreply.github.com>
Co-Authored-By: Claude Fable 5 <noreply@anthropic.com>
Parts:
- moved M1 31.4 mm to (245.7, 9.39)
- moved U3 28.4 mm to (228.6, 9.39)
- moved M3 25.5 mm to (265.7, 46.8)
- moved U6 25.5 mm to (250.6, 46.8)
- moved U2 25.5 mm to (226.6, 46.8)
- moved U5 21.8 mm to (189.9, 60.8)
- moved C3 16.9 mm to (164.1, 60.8)
- moved C2 15.8 mm to (174.9, 9.40)
- moved SR1 15.0 mm to (143.0, 60.8)
- moved U1 13.3 mm to (159.3, 9.40)
- moved M2 13.2 mm to (124.3, 60.8)
- moved SOL1 11.7 mm to (124.3, 32.9)
- moved U4 11.0 mm to (138.9, 32.9)
- moved C1 10.8 mm to (143.7, 9.40)
- moved J1 10.6 mm to (129.7, 9.40)
Connections:
- SR1 pad 3: GND -> +12V
- U1 pad 1: +12V -> (no net)
- U1 pad 2: GND -> +12V
- U1 pad 3: +5V -> +12V
- U1 pad 4: +12V -> GND
- U3 pad 3: I2C_SDA -> I2C_SCL
- U3 pad 4: I2C_SCL -> I2C_SDA
- U3 pad 6: HAPT_EN -> VIB_A
- U3 pad 7: VIB_A -> VIB_B
- U3 pad 8: VIB_B -> (no net)
- U4 pad 1: +12V -> SOL_B
- U4 pad 2: GND -> SOL_A
- U4 pad 3: SOL_A -> +12V
- U4 pad 4: SOL_B -> GND
- U4 pad 5: SOL_IN1 -> SOL_IN2
- U4 pad 6: SOL_IN2 -> SOL_IN1
- U4 pad 7: GND -> +12V
- U5 pad 11: STP_A1 -> (no net)
- U5 pad 12: STP_A2 -> (no net)
- U5 pad 13: STP_B1 -> GND
- U5 pad 14: STP_B2 -> GND
- U5 pad 3: STP_RX -> (no net)
- U5 pad 4: STP_TX -> (no net)
- U5 pad 5: (no net) -> GND
- U5 pad 6: (no net) -> STP_RX
- U5 pad 7: GND -> STP_TX
- U5 pad 9: +12V -> (no net)
Other:
- board size 100 x 100 mm -> 110 x 110 mm

Commit message: Add second dispensing-angle servo M4 (SERVO_SIG2 on GP2) — 2-servo design alignment
williamulbz's PR #76 review flagged that the board predates the move to
the 2-servo design (PR #66 dual-servo hinge; PR #100 generate.py rev C).
build_starter_board.py now emits a second 3-pin servo header M4 wired
exactly as rev C: SIG -> SERVO_SIG2 on Pico GP2 (mirrored in firmware via
config.SERVO2_INVERT), +5V/GND shared. M4 joins the logic/mcu placement
cluster beside M3, edge-biased for cable exit.

Counts: 16 footprints / 175 pads / 99 net-assigned / 23 nets (placed
outline ~162x85 mm; unplaced stays 110x110 mm at ~51% courtyard).
Verified: kicad-cli netlist 99 pins / 23 nets / zero unconnected on both
trios (SERVO_SIG2 = M4.3 <-> U2.4/GP2), pcbnew DRC clean (no courtyard/
clearance/short errors), 16<->16 footprint<->symbol UUID bijection,
byte-for-byte reproducible, KiCad 7 20221018 format kept. Both trios +
previews + summary regenerated; note 21 update block, note 24 superseded
caveat (run-2 candidates lack M4; +5V now wants 2000 mA in Quilter), and
background README updated.

Co-authored-by: Sterling G. Baird <45469701+sgbaird@users.noreply.github.com>
Co-Authored-By: Claude Fable 5 <noreply@anthropic.com>
Parts:
- added M4: Servo_3pin, Connector_PinHeader_2.54mm:PinHeader_1x03_P2.54mm_Vertical, F.Cu at (271.9, 46.8)
Connections:
- U2 pad 4: (no net) -> SERVO_SIG2
